File: KiCadFiles/brownberryKeeb.kicad_pcb (KiCad board)
At the start: 2 copper layers, 140 x 65 mm, 86 parts, among them SW1 Q, SW10 D, SW11 C, SW12 META, SW13 R, SW14 F, SW15 V, SW16 SHIFT, SW17 T, SW18 G, SW19 B, SW2 A, SW20 SPACE, SW21 Y, SW22 H, SW23 N, SW24 FN1, SW25 U, SW26 J, SW27 M, SW28 FN2, SW29 I, SW3 Z, SW30 K, SW31 ,, SW32 HOME, SW33 O, SW34 L, SW35 ., SW36 END, SW37 P, SW38 ;, SW39 /, SW4 CTRL, SW40 BACKSPACE, SW5 W, SW6 S, SW7 X, SW8 ALT, SW9 E, U1 Pico

Commit message: fixed PCB forgotten trace and added my homebrew footprints
Routing:
- net COL8: track 36.1 -> 40.4 mm
Changed lines of the file:
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@@
+	)
+	(segment
+		(start 175.86434 121.889213)
+		(end 176.114342 122.139215)
+		(width 0.2)
+		(layer "F.Cu")
+		(net 53)
 	)
 	(segment
@@
 		(width 0.2)
 		(layer "F.Cu")
+		(net 53)
+	)
+	(segment
+		(start 175.86434 117.889217)
+		(end 175.86434 121.889213)
+		(width 0.2)
+		(layer "F.Cu")
